File: power_supply_buck/power_supply_buck.kicad_sch (KiCad schematic)
At the start: 0 parts

Commit message: footprint
Parts:
- added U1: AP63203WU-7, AP63203WU-7_DIO, symbol AP63203:AP63203WU-7

Commit message: power supply
Parts:
- added C1, C2: 10uf, Capacitor_SMD:C_1210_3225Metric_Pad1.33x2.70mm_HandSolder, symbol Device:C
- added C3: 100nf, Capacitor_SMD:C_0805_2012Metric_Pad1.18x1.45mm_HandSolder, symbol Device:C
- added C4, C5: 22uf, Capacitor_SMD:C_1210_3225Metric_Pad1.33x2.70mm_HandSolder, symbol Device:C
- added C6: 100uf, Capacitor_SMD:C_Elec_6.3x7.7, symbol Device:C_Polarized
- added J1: Conn_01x02_Pin, symbol Connector:Conn_01x02_Pin
- added L1: 4.7uH, Inductor_SMD:L_Bourns_SRR1260, symbol Device:L
Connections:
- net +3.3V: now also U1.1 (FB), C4.1, C5.1, L1.2
- net GND: now also U1.4 (GND), C1.2, C2.2, C4.2, C5.2, C6.2
- net VCC: now also U1.3 (VIN), C1.1, C2.1, C6.1
- net at U1.5 (SW): now also C3.2, L1.1
- net at U1.6 (BST): now also C3.1
Other:
- moved on the sheet: U1

Commit message: done buck sch
Parts:
- added J2: VOUT, Connector_PinHeader_2.54mm:PinHeader_1x02_P2.54mm_Vertical, symbol Connector:Conn_01x02_Pin
- added J3: VIN+, Connector_PinHeader_1.00mm:PinHeader_1x01_P1.00mm_Vertical, symbol Connector:Conn_01x01_Pin
- added J4: EN, Connector_PinHeader_1.00mm:PinHeader_1x01_P1.00mm_Vertical, symbol Connector:Conn_01x01_Pin
- added J5: VOUT+, Connector_PinHeader_1.00mm:PinHeader_1x01_P1.00mm_Vertical, symbol Connector:Conn_01x01_Pin
- added J6, J7: GND, Connector_PinHeader_1.00mm:PinHeader_1x01_P1.00mm_Vertical, symbol Connector:Conn_01x01_Pin
- added TP1: VIN+, TestPoint:TestPoint_Pad_1.0x1.0mm, symbol Connector:TestPoint
- added TP2: EN, TestPoint:TestPoint_Pad_1.0x1.0mm, symbol Connector:TestPoint
- added TP3: VOUT+, TestPoint:TestPoint_Pad_1.0x1.0mm, symbol Connector:TestPoint
- added TP4, TP5: GND, TestPoint:TestPoint_Pad_1.0x1.0mm, symbol Connector:TestPoint
- J1: value Conn_01x02_Pin -> VIN; footprint (none) -> Connector_PinHeader_2.54mm:PinHeader_1x02_P2.54mm_Vertical
Connections:
- net +3.3V: now also TP3.1
- net GND: now also J1.2 (Pin_2), J7.1 (Pin_1), TP4.1, TP5.1
- net VCC: now also J1.1 (Pin_1), J3.1 (Pin_1), TP1.1
- net at U1.2 (EN): now also J4.1 (Pin_1), TP2.1
Other:
- moved on the sheet: J1

Commit message: done sch
Connections:
- net +3.3V is gone; now on an unnamed net: C4.1, C5.1, L1.2, TP3.1, U1.1 (FB)
- net GND: now also J2.1 (Pin_1), J6.1 (Pin_1)
- net at J2.2 (Pin_2): now also J5.1 (Pin_1)
Other:
- moved on the sheet: J2, J5, J6

Commit message: done
Parts:
- U1: footprint AP63203WU-7_DIO -> (none)
Changed lines of the file:
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@@
 			)
 		)
-		(property "Footprint" "AP63203WU-7_DIO"
+		(property "Footprint" ""
 			(at 130.81 90.17 0)
 			(effects

Commit message: no footprint :(
Parts:
- U1: footprint (none) -> AP63203WU-7_DIO
Changed lines of the file:
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@@
 			)
 		)
-		(property "Footprint" ""
+		(property "Footprint" "AP63203WU-7_DIO"
 			(at 130.81 90.17 0)
 			(effects

Commit message: footprint
Parts:
- U1: footprint AP63203WU-7_DIO -> AP63203.footprints:AP63203WU-7_DIO
Changed lines of the file:
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@@
 			)
 		)
-		(property "Footprint" "AP63203WU-7_DIO"
+		(property "Footprint" "AP63203.footprints:AP63203WU-7_DIO"
 			(at 130.81 90.17 0)
 			(effects

Commit message: routing
Parts:
- U1: value AP63203WU-7 -> AP63203WU
Changed lines of the file:
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@@
 			)
 		)
-		(property "Value" "AP63203WU-7"
+		(property "Value" "AP63203WU"
 			(at 151.13 82.55 0)
 			(effects
